Commit message: zadanie 3 changes

File: custom_urdf/urdf/custom.urdf (robot description, URDF)
Before this commit: robot custom_urdf, 6 links, 5 joints
Links:
- added link connector
Joints:
- added joint wrist_connector: type prismatic, parent connector, child hand, origin xyz=0.0 0 0.0 rpy=0.0 1.578 0, limit lower=0.0 upper=0.5 effort=1000.0 velocity=0.5
- joint fixed_end: origin xyz=0 0 0.5 rpy=0 0 0 -> xyz=-0.5 0 0 rpy=0 0 0
- joint wrist: child hand -> connector

File: install/custom_urdf/share/custom_urdf/custom.urdf (robot description, URDF)
Before this commit: robot planar_3dof, 6 links, 5 joints
Links:
- added link connector
Joints:
- added joint wrist_connector: type prismatic, parent connector, child hand, origin xyz=0.0 0 0.0 rpy=0.0 1.578 0, limit lower=0.0 upper=0.5 effort=1000.0 velocity=0.5
- joint elbow: origin xyz=0.5 0.0 0.0 rpy=0.0 0.0 0.0 -> xyz=0.5 0.0 0.0 rpy=0.0 0 0.0
- joint fixed_end: origin xyz=0.0 0.0 0.5 rpy=0.0 0.0 0.0 -> xyz=-0.5 0 0 rpy=0 0 0
- joint shoulder: origin xyz=0.0 0.0 1.3 rpy=0.0 0.0 0.0 -> xyz=0 0 1.3 rpy=0 0 0
- joint wrist: child hand -> connector; origin xyz=0.5 0.0 0.0 rpy=-3.14 0.0 0.0 -> xyz=0.5 0 0 rpy=-3.14 0 0
