Commit message: added new xacro

File: custom_urdf/urdf/custom.urdf.xacro (robot description, xacro)
@@ -7,4 +7,5 @@
   <xacro:property name="joint_wrist_params" value="${joint_params['calc_params']['ros__parameters']['joint_wrist']}" />
   <xacro:property name="joint_fixed_end_params" value="${joint_params['calc_params']['ros__parameters']['joint_fixed_end']}" />
+  <xacro:property name="joint_wrist_connector_params" value="${joint_params['calc_params']['ros__parameters']['joint_wrist_connector']}" />
   <xacro:property name="joint_shoulder_origin_xyz" value="${joint_shoulder_params[0]} ${joint_shoulder_params[1]} ${joint_shoulder_params[2]}" />
   <xacro:property name="joint_shoulder_origin_rpy" value="${joint_shoulder_params[3]} ${joint_shoulder_params[4]} ${joint_shoulder_params[5]}" />
@@ -14,5 +15,5 @@
   <xacro:property name="joint_elbow_axis" value="${int(joint_elbow_params[6])} ${int(joint_elbow_params[7])} ${int(joint_elbow_params[8])}" />
   <xacro:property name="joint_wrist_origin_xyz" value="${joint_wrist_params[0]} ${joint_wrist_params[1]} ${joint_wrist_params[2]}" />
-  <xacro:property name="joint_wrist_origin_rpy" value="${joint_wrist_params[3]} ${joint_wrist_params[4]} ${joint_wrist_params[5]}" />
+  <xacro:property name="joint_wrist_origin_rpy" value="-3.14 0 0" />
   <xacro:property name="joint_wrist_axis" value="${int(joint_wrist_params[6])} ${int(joint_wrist_params[7])} ${int(joint_wrist_params[8])}" />
   <xacro:property name="joint_fixed_end_origin_xyz" value="${joint_fixed_end_params[0]} ${joint_fixed_end_params[1]} ${joint_fixed_end_params[2]}" />
@@ -29,9 +30,11 @@
   <xacro:property name="link_forearm_rpy" value="0 1.5708 0" />
   <xacro:property name="link_forearm_length" value="${joint_wrist_params[0]}" />
-  <xacro:property name="link_hand_xyz1" value="${joint_fixed_end_params[0]/2} ${joint_fixed_end_params[1]/2} ${joint_fixed_end_params[2]/2}" />
-  <xacro:property name="link_hand_xyz2" value="${joint_fixed_end_params[2]/2} ${joint_fixed_end_params[1]/2} ${joint_fixed_end_params[0]/2}" />
-  <xacro:property name="link_hand_rpy1" value="0 0 1.5708" />
-  <xacro:property name="link_hand_rpy2" value="0 1.5708 0" />
-  <xacro:property name="link_hand_length" value="${joint_fixed_end_params[2]}" />
+  <xacro:property name="link_hand_xyz" value="${joint_fixed_end_params[0]/2} ${joint_fixed_end_params[1]/2} ${joint_fixed_end_params[2]/2}" />
+  <xacro:property name="link_hand_rpy" value="${joint_wrist_connector_params[3]} ${joint_wrist_connector_params[4]} ${joint_wrist_connector_params[5]}" />
+  <xacro:property name="link_hand_length" value="${-joint_fixed_end_params[0]}" />
+  <xacro:property name="joint_wrist_connector_origin_xyz" value="${joint_wrist_connector_params[0]} ${joint_wrist_connector_params[1]} ${joint_wrist_connector_params[2]}" />
+  <xacro:property name="joint_wrist_connector_origin_rpy" value="${joint_wrist_connector_params[3]} ${joint_wrist_connector_params[4]} ${joint_wrist_connector_params[5]}" />
+  <xacro:property name="joint_wrist_connector_axis" value="${joint_wrist_connector_params[6]} ${joint_wrist_connector_params[7]} ${joint_wrist_connector_params[8]}" />
+  <xacro:property name="joint_wrist_connector_upperlimit" value="${link_hand_length}" />
   <material name="red">
     <color rgba="0.8 0.0 0.0 1.0"/>
@@ -78,5 +81,5 @@
     </link>
   </xacro:macro>
-    <xacro:macro name="joint_template" params="name type parent child xyz rpy axis">
+    <xacro:macro name="joint_template" params="name type parent child xyz rpy axis prismatic_limit">
     <joint name="${name}" type="${type}">
       <parent link="${parent}" />
@@ -86,4 +89,7 @@
       <axis xyz="${axis}" />
       <limit lower="-1.57" upper="1.57" effort="0" velocity="0.5" />
+    </xacro:if>
+      <xacro:if value="${type == 'prismatic'}">
+      <limit lower="0.0" upper="${prismatic_limit}" effort="1000.0" velocity="0.5" />
     </xacro:if>
     </joint>
@@ -112,8 +118,8 @@
   </link>
   </xacro:macro>
-  <xacro:macro name="hand_template" params="name xyz1 xyz2 rpy1 rpy2 length radius material" >
+  <xacro:macro name="hand_template" params="name xyz rpy length radius material" >
     <link name="${name}">
     <visual>
-      <origin xyz="${xyz1}" rpy="${rpy1}" />
+      <origin xyz="${xyz}" rpy="${rpy}" />
       <geometry>
         <cylinder length="${length}" radius="${radius}" />
@@ -122,5 +128,5 @@
     </visual>
     <collision>
-      <origin rpy="${rpy2}" xyz="${xyz2}" />
+      <origin rpy="${rpy}" xyz="${xyz}" />
       <geometry>
         <cylinder length="${length}" radius="${radius}" />
@@ -129,5 +135,5 @@
     </collision>
     <inertial>
-      <origin xyz="${xyz1}" rpy="${rpy2}" />
+      <origin xyz="${xyz}" rpy="${rpy}" />
       <mass value="1" />
       <inertia ixx="1.0" ixy="0.0" ixz="0.0" iyy="1.0" iyz="0.0" izz="1.0" />
@@ -142,9 +148,11 @@
   </joint>
   <link_template name="arm" rpy="${link_arm_rpy}" xyz="${link_arm_xyz}" length="${link_arm_length}" radius="0.05" material="red" />
-  <joint_template name="shoulder" type="revolute" parent="body" child="arm" xyz="${joint_shoulder_origin_xyz}" rpy="${joint_shoulder_origin_rpy}" axis="${joint_shoulder_axis}" />
+  <joint_template name="shoulder" type="revolute" parent="body" child="arm" xyz="${joint_shoulder_origin_xyz}" rpy="${joint_shoulder_origin_rpy}" axis="${joint_shoulder_axis}" prismatic_limit="none"/>
   <link_template name="forearm" rpy="${link_forearm_rpy}" xyz="${link_forearm_xyz}" length="${link_forearm_length}" radius="0.05" material="grey" />
-  <joint_template name="elbow" type="revolute" parent="arm" child="forearm" xyz="${joint_elbow_origin_xyz}" rpy="${joint_elbow_origin_rpy}" axis="${joint_elbow_axis}" />
-  <hand_template name="hand" xyz1="${link_hand_xyz1}" xyz2="${link_hand_xyz2}" rpy1="${link_hand_rpy1}" rpy2="${link_hand_rpy2}" length="${link_hand_length}" radius="0.05" material="red" />
-  <joint_template name="wrist" type="fixed" parent="forearm" child="hand" xyz="${joint_wrist_origin_xyz}" rpy="${joint_wrist_origin_rpy}" axis="${joint_wrist_axis}" />
+  <joint_template name="elbow" type="revolute" parent="arm" child="forearm" xyz="${joint_elbow_origin_xyz}" rpy="${joint_elbow_origin_rpy}" axis="${joint_elbow_axis}" prismatic_limit="none"/>
+  <hand_template name="hand" xyz="${link_hand_xyz}" rpy="${link_hand_rpy}" length="${link_hand_length}" radius="0.05" material="red" />
+  <link name="connector" />
+  <joint_template name="wrist" type="fixed" parent="forearm" child="connector" xyz="${joint_wrist_origin_xyz}" rpy="${joint_wrist_origin_rpy}" axis="${joint_wrist_axis}" prismatic_limit="none"/>
+   <joint_template name="wrist_connector" type="prismatic" parent="connector" child="hand" xyz="${joint_wrist_connector_origin_xyz}" rpy="${joint_wrist_connector_origin_rpy}" axis="${joint_wrist_connector_axis}" prismatic_limit="${joint_wrist_connector_upperlimit}"/>
 <link name="end">
     <visual>
@@ -168,4 +176,4 @@
     </inertial>
   </link>
-  <joint_template name="fixed_end" type="fixed" parent="hand" child="end" xyz="${joint_fixed_end_origin_xyz}" rpy="${joint_fixed_end_origin_rpy}" axis="${joint_fixed_end_axis}" />
+  <joint_template name="fixed_end" type="fixed" parent="hand" child="end" xyz="${joint_fixed_end_origin_xyz}" rpy="${joint_fixed_end_origin_rpy}" axis="${joint_fixed_end_axis}" prismatic_limit="none"/>
 </robot>

File: install/custom_urdf/share/custom_urdf/custom.urdf (robot description, URDF)
Before this commit: robot custom_urdf, 7 links, 6 joints
Links:
- link arm: geometry collision cylinder length=2.0 radius=0.05; visual cylinder length=2.0 radius=0.05
- link body: geometry collision cylinder length=5.0 radius=0.075; visual cylinder length=5.0 radius=0.075
- link forearm: geometry collision cylinder length=3.0 radius=0.05; visual cylinder length=3.0 radius=0.05
- link hand: geometry collision cylinder length=3.0 radius=0.05; visual cylinder length=3.0 radius=0.05
Joints:
- joint elbow: origin xyz=0.5 0.0 0.0 rpy=0.0 0 0.0 -> xyz=2.0 0.0 0.0 rpy=0.0 0.0 0.0
- joint fixed_end: origin xyz=-0.5 0 0 rpy=0 0 0 -> xyz=-3.0 0.0 0.0 rpy=0.0 0.0 0.0
- joint shoulder: origin xyz=0 0 1.3 rpy=0 0 0 -> xyz=0.0 0.0 5.0 rpy=0.0 0.0 0.0
- joint wrist: origin xyz=0.5 0 0 rpy=-3.14 0 0 -> xyz=3.0 0.0 0.0 rpy=-3.14 0 0
- joint wrist_connector: limit lower=0.0 upper=0.5 effort=1000.0 velocity=0.5 -> lower=0.0 upper=3.0 effort=1000.0 velocity=0.5; origin xyz=0.0 0 0.0 rpy=0.0 1.578 0 -> xyz=0.0 0.0 0.0 rpy=0.0 1.578 0.0

Commit message: New changes

File: custom_urdf/urdf/custom.urdf.xacro (robot description, xacro)
@@ -88,5 +88,10 @@
       <xacro:if value="${type == 'revolute'}">
       <axis xyz="${axis}" />
-      <limit lower="-1.57" upper="1.57" effort="0" velocity="0.5" />
+      <xacro:if value="${name == 'shoulder'}">
+      	<limit lower="-3.14" upper="3.14" effort="0" velocity="0.5" />
+      </xacro:if>
+    	<xacro:if value="${name == 'elbow'}">
+      	<limit lower="-1.57" upper="1.57" effort="0" velocity="0.5" />
+      </xacro:if>
     </xacro:if>
       <xacro:if value="${type == 'prismatic'}">

File: install/custom_urdf/share/custom_urdf/custom.urdf (robot description, URDF)
Before this commit: robot planar_3dof, 7 links, 6 joints
Joints:
- joint shoulder: limit lower=-1.57 upper=1.57 effort=0 velocity=0.5 -> lower=-3.14 upper=3.14 effort=0 velocity=0.5
