Commit message: final changes

File: install/custom_urdf/share/custom_urdf/custom.urdf (robot description, URDF)
Before this commit: robot custom_urdf, 6 links, 5 joints
Joints:
- joint elbow: origin xyz=0.5 0.0 0.0 rpy=0.0 0 0.0 -> xyz=0.5 0.0 0.0 rpy=0.0 0.0 0.0
- joint fixed_end: origin xyz=0 0 0.5 rpy=0 0 0 -> xyz=0.0 0.0 0.5 rpy=0.0 0.0 0.0
- joint shoulder: origin xyz=0 0 1.3 rpy=0 0 0 -> xyz=0.0 0.0 1.3 rpy=0.0 0.0 0.0
- joint wrist: origin xyz=0.5 0 0 rpy=-3.14 0 0 -> xyz=0.5 0.0 0.0 rpy=-3.14 0.0 0.0

Commit message: Final version of NONKDL node

File: install/custom_urdf/share/custom_urdf/custom.urdf (robot description, URDF)
Before this commit: robot planar_3dof, 7 links, 6 joints
Links:
- link arm: geometry collision cylinder length=0.5 radius=0.05; visual cylinder length=0.5 radius=0.05
- link body: geometry collision cylinder length=1.5 radius=0.075; visual cylinder length=1.5 radius=0.075
- link forearm: geometry collision cylinder length=0.5 radius=0.05; visual cylinder length=0.5 radius=0.05
- link hand: geometry collision cylinder length=0.5 radius=0.05; visual cylinder length=0.5 radius=0.05
Joints:
- joint elbow: origin xyz=2.0 0.0 0.0 rpy=0.0 0.0 0.0 -> xyz=0.5 0.0 0.0 rpy=0.0 0.0 0.0
- joint fixed_end: origin xyz=-3.0 0.0 0.0 rpy=0.0 0.0 0.0 -> xyz=-0.5 0.0 0.0 rpy=0.0 0.0 0.0
- joint shoulder: origin xyz=0.0 0.0 5.0 rpy=0.0 0.0 0.0 -> xyz=0.0 0.0 1.5 rpy=0.0 0.0 0.0
- joint wrist: origin xyz=3.0 0.0 0.0 rpy=-3.14 0 0 -> xyz=0.5 0.0 0.0 rpy=-3.14 0 0
- joint wrist_connector: limit lower=0.0 upper=3.0 effort=1000.0 velocity=0.5 -> lower=0.0 upper=0.5 effort=1000.0 velocity=0.5
